Commit message: from linux

File: ROS/catkin_ws/src/cat_vehicle_pkgs/azcar_sim/urdf/azcar.xacro (robot description, xacro)
@@ -31,5 +31,5 @@
 <robot name="$(arg roboname)" xmlns:xacro="http://www.ros.org/wiki/xacro">
   <xacro:property name="PI" value="3.1415926835897931"/>
-<!--  <xacro:property name="base_height" value="0"/> -->
+  <!--  <xacro:property name="base_height" value="0"/> -->
   <xacro:property name="base_height" value="1.0639"/>
   <xacro:property name="base_mass" value="2050"/>
@@ -58,256 +58,256 @@
   <xacro:property name="car_width" value="1.301"/>
   <xacro:property name="tyre_origin">
-	<origin xyz="0 0 0" rpy="${PI/2} 0 0"/>
+    <origin xyz="0 0 0" rpy="${PI/2} 0 0"/>
   </xacro:property>
   <xacro:property name="tyre_origin_2">
-        <origin xyz="0 0 0" rpy="0 0 ${PI/2}"/>
+    <origin xyz="0 0 0" rpy="0 0 ${PI/2}"/>
   </xacro:property>
   <xacro:property name="tyre_origin_3">
-        <origin xyz="0 0 0" rpy="0 0 ${-PI/2}"/>
+    <origin xyz="0 0 0" rpy="0 0 ${-PI/2}"/>
   </xacro:property>
-	<xacro:include filename="$(find azcar_sim)/urdf/azcar_slipping.gazebo"/>
-<!--Car Body-->
-<link name="base_link">
-    <collision>
-         <origin xyz="0 0 ${base_height}" rpy="0 0 0"/>
-           <geometry>
-            <box size="2.62 ${car_width} ${car_height}"/>
-        </geometry>
-      </collision>
-     <visual>
-        <origin xyz="-0.25 0 ${base_height + 0.05}" rpy="0 0 0"/>
-        <geometry>
-          <mesh filename="package://azcar_sim/meshes/ford_escape_no_wheels_2.dae"/>
-        </geometry>
-     </visual>
-</link>
-<joint name="inertial_joint" type="fixed">
-      <parent link="base_link"/>
-      <child link="main_mass"/>
-      <origin xyz="0 0 0" rpy="0 0 0"/>
-</joint>
-<link name="main_mass" type="fixed">
-     <parent link="inertial_joint"/>
-     <inertial>
-        <origin xyz="0 0 ${base_height}" rpy="0 0 0"/>
-        <mass value="${base_mass}"/>
-        <inertia
+  <xacro:include filename="$(find azcar_sim)/urdf/azcar_slipping.gazebo"/>
+  <!--Car Body-->
+  <link name="base_link">
+    <collision>
+      <origin xyz="0 0 ${base_height}" rpy="0 0 0"/>
+      <geometry>
+        <box size="2.62 ${car_width} ${car_height}"/>
+      </geometry>
+    </collision>
+    <visual>
+      <origin xyz="-0.25 0 ${base_height + 0.05}" rpy="0 0 0"/>
+      <geometry>
+        <mesh filename="package://azcar_sim/meshes/ford_escape_no_wheels_2.dae"/>
+      </geometry>
+    </visual>
+  </link>
+  <joint name="inertial_joint" type="fixed">
+    <parent link="base_link"/>
+    <child link="main_mass"/>
+    <origin xyz="0 0 0" rpy="0 0 0"/>
+  </joint>
+  <link name="main_mass" type="fixed">
+    <parent link="inertial_joint"/>
+    <inertial>
+      <origin xyz="0 0 ${base_height}" rpy="0 0 0"/>
+      <mass value="${base_mass}"/>
+      <inertia
           ixx="${base_mass_ixx}"  ixy="0.000000" ixz="${base_mass_ixz}"
           iyy="${base_mass_iyy}" iyz="0.000000"
           izz="${base_mass_izz}"/>
-      </inertial>
-</link>
-<!--Back Right Wheel-->
-<joint name="back_right_wheel_joint" type="continuous">
-      <parent link="base_link"/>
-      <child link="back_right_wheel_link"/>
-      <origin xyz="${-tyre_x} ${-tyre_y} ${tyre_r}" rpy="0 0 0"/>
-      <axis xyz="0 1 0"/>
-      <dynamics damping="0.1"/>
-     <limit effort="10000" velocity="100" />
-      <joint_properties damping="0.0" friction="0.0" />
-</joint>
-<link name="back_right_wheel_link">
-     <collision>
-      <xacro:insert_block name="tyre_origin"/>
-        <geometry>
-         <cylinder length="${tyre_length}" radius="${tyre_radius}"/>
-        </geometry>
-     </collision>
-     <visual>
+    </inertial>
+  </link>
+  <!--Back Right Wheel-->
+  <joint name="back_right_wheel_joint" type="continuous">
+    <parent link="base_link"/>
+    <child link="back_right_wheel_link"/>
+    <origin xyz="${-tyre_x} ${-tyre_y} ${tyre_r}" rpy="0 0 0"/>
+    <axis xyz="0 1 0"/>
+    <dynamics damping="0.1"/>
+    <limit effort="10000" velocity="100" />
+    <joint_properties damping="0.0" friction="0.0" />
+  </joint>
+  <link name="back_right_wheel_link">
+    <collision>
+      <xacro:insert_block name="tyre_origin"/>
+      <geometry>
+        <cylinder length="${tyre_length}" radius="${tyre_radius}"/>
+      </geometry>
+    </collision>
+    <visual>
       <xacro:insert_block name="tyre_origin_3"/>
-        <geometry>
-          <mesh filename="package://azcar_sim/meshes/ford_escape_wheel.dae"/>
-      <scale xyz="1.2 1 1"/>
-        </geometry>
-      </visual>
-      <inertial>
-        <origin xyz="0 0 0" rpy="0 0 0"/>
-        <mass value="${tyre_mass}"/>
-        <inertia
+      <geometry>
+        <mesh filename="package://azcar_sim/meshes/ford_escape_wheel.dae"/>
+        <scale xyz="1.2 1 1"/>
+      </geometry>
+    </visual>
+    <inertial>
+      <origin xyz="0 0 0" rpy="0 0 0"/>
+      <mass value="${tyre_mass}"/>
+      <inertia
           ixx="${tyre_mass_ixx}"  ixy="0.000000"  ixz="0.000000"
           iyy="${tyre_mass_iyy}"  iyz="0.000000"
           izz="${tyre_mass_izz}"/>
-      </inertial>
-</link>
-<!--Back Left Wheel-->
-<joint name="back_left_wheel_joint" type="continuous">
-      <parent link="base_link"/>
-      <child link="back_left_wheel_link"/>
-      <origin xyz="${-tyre_x} ${tyre_y} ${tyre_r}" rpy="0 0 0"/>
-      <axis xyz="0 1 0"/>
-      <dynamics damping="0.1"/>
-      <limit effort="10000" velocity="100" />
-      <joint_properties damping="0.0" friction="0.0" />
-</joint>
-<link name="back_left_wheel_link">
-     <collision>
-      <xacro:insert_block name="tyre_origin"/>
-        <geometry>
-         <cylinder length="0.229" radius="${tyre_radius}"/>
-        </geometry>
-     </collision>
-     <visual>
+    </inertial>
+  </link>
+  <!--Back Left Wheel-->
+  <joint name="back_left_wheel_joint" type="continuous">
+    <parent link="base_link"/>
+    <child link="back_left_wheel_link"/>
+    <origin xyz="${-tyre_x} ${tyre_y} ${tyre_r}" rpy="0 0 0"/>
+    <axis xyz="0 1 0"/>
+    <dynamics damping="0.1"/>
+    <limit effort="10000" velocity="100" />
+    <joint_properties damping="0.0" friction="0.0" />
+  </joint>
+  <link name="back_left_wheel_link">
+    <collision>
+      <xacro:insert_block name="tyre_origin"/>
+      <geometry>
+        <cylinder length="0.229" radius="${tyre_radius}"/>
+      </geometry>
+    </collision>
+    <visual>
       <xacro:insert_block name="tyre_origin_2"/>
-        <geometry>
-          <mesh filename="package://azcar_sim/meshes/ford_escape_wheel.dae"/>
-          <scale xyz="1.2 1 1"/>
-        </geometry>
-      </visual>
-      <inertial>
-        <origin xyz="0 0 0" rpy="0 0 0"/>
-        <mass value="${tyre_mass}"/>
-        <inertia
+      <geometry>
+        <mesh filename="package://azcar_sim/meshes/ford_escape_wheel.dae"/>
+        <scale xyz="1.2 1 1"/>
+      </geometry>
+    </visual>
+    <inertial>
+      <origin xyz="0 0 0" rpy="0 0 0"/>
+      <mass value="${tyre_mass}"/>
+      <inertia
           ixx="${tyre_mass_ixx}"  ixy="0.000000"  ixz="0.000000"
           iyy="${tyre_mass_iyy}"  iyz="0.000000"
           izz="${tyre_mass_izz}"/>
-      </inertial>
-</link>
-<!--Right Steering-->
-<joint name="front_right_steering_joint" type="revolute">
-	<parent link="base_link"/>
-	<child link="front_right_steering_link"/>
-	<origin xyz="${tyre_x} ${-car_width/2 - str_length/2} ${tyre_r}" rpy="0 0 0"/>
-        <axis xyz="0 0 1"/>
-	<limit effort="1000.0" lower="${-str_angle}" upper="${str_angle}" velocity="0.5"/>
-</joint>
-<link name="front_right_steering_link">
-	<collision>
-	      <xacro:insert_block name="tyre_origin"/>
-	        <geometry>
-        	 <cylinder length="${str_length}" radius="${str_radius}"/>
-       		</geometry>
-	</collision>
-	<visual>
-              <xacro:insert_block name="tyre_origin"/>
-                <geometry>
-                 <cylinder length="${str_length}" radius="${str_radius}"/>
-                </geometry>
-	</visual>
-      <inertial>
-        <origin xyz="0 0 0" rpy="0 0 0"/>
-        <mass value="10.00"/>
-        <inertia
+    </inertial>
+  </link>
+  <!--Right Steering-->
+  <joint name="front_right_steering_joint" type="revolute">
+    <parent link="base_link"/>
+    <child link="front_right_steering_link"/>
+    <origin xyz="${tyre_x} ${-car_width/2 - str_length/2} ${tyre_r}" rpy="0 0 0"/>
+    <axis xyz="0 0 1"/>
+    <limit effort="1000.0" lower="${-str_angle}" upper="${str_angle}" velocity="0.5"/>
+  </joint>
+  <link name="front_right_steering_link">
+    <collision>
+      <xacro:insert_block name="tyre_origin"/>
+      <geometry>
+        <cylinder length="${str_length}" radius="${str_radius}"/>
+      </geometry>
+    </collision>
+    <visual>
+      <xacro:insert_block name="tyre_origin"/>
+      <geometry>
+        <cylinder length="${str_length}" radius="${str_radius}"/>
+      </geometry>
+    </visual>
+    <inertial>
+      <origin xyz="0 0 0" rpy="0 0 0"/>
+      <mass value="10.00"/>
+      <inertia
           ixx="0.4"  ixy="0.000000"  ixz="0.000000"
           iyy="0.6"  iyz="0.000000"
           izz="0.4"/>
-      </inertial>
-</link>
-<!--Right Front Wheel-->
-<joint name="front_right_wheel_joint" type="continuous">
-      <parent link="front_right_steering_link"/>
-      <child link="front_right_wheel_link"/>
-      <origin xyz="0 ${-str_length/2 - tyre_length/2} 0" rpy="0 0 0"/>
-      <axis xyz="0 1 0"/>
-</joint>
-<link name="front_right_wheel_link">
-     <collision>
-      <xacro:insert_block name="tyre_origin"/>
-        <geometry>
-         <cylinder length="${tyre_length}" radius="${tyre_radius}"/>
-	</geometry>
-     </collision>
-     <visual>
+    </inertial>
+  </link>
+  <!--Right Front Wheel-->
+  <joint name="front_right_wheel_joint" type="continuous">
+    <parent link="front_right_steering_link"/>
+    <child link="front_right_wheel_link"/>
+    <origin xyz="0 ${-str_length/2 - tyre_length/2} 0" rpy="0 0 0"/>
+    <axis xyz="0 1 0"/>
+  </joint>
+  <link name="front_right_wheel_link">
+    <collision>
+      <xacro:insert_block name="tyre_origin"/>
+      <geometry>
+        <cylinder length="${tyre_length}" radius="${tyre_radius}"/>
+      </geometry>
+    </collision>
+    <visual>
       <xacro:insert_block name="tyre_origin_3"/>
-        <geometry>
-          <mesh filename="package://azcar_sim/meshes/ford_escape_wheel.dae"/>
+      <geometry>
+        <mesh filename="package://azcar_sim/meshes/ford_escape_wheel.dae"/>
         <scale xyz="1.2 1 1"/>
-       </geometry>
-      </visual>
-      <inertial>
-        <origin xyz="0 0 0" rpy="0 0 0"/>
-        <mass value="${tyre_mass}"/>
-        <inertia
+      </geometry>
+    </visual>
+    <inertial>
+      <origin xyz="0 0 0" rpy="0 0 0"/>
+      <mass value="${tyre_mass}"/>
+      <inertia
           ixx="${tyre_mass_ixx}"  ixy="0.000000"  ixz="0.000000"
           iyy="${tyre_mass_iyy}"  iyz="0.000000"
           izz="${tyre_mass_izz}"/>
-      </inertial>
-</link>
-<!--Left Steering-->
-<joint name="front_left_steering_joint" type="revolute">
-        <parent link="base_link"/>
-        <child link="front_left_steering_link"/>
-        <origin xyz="${tyre_x} ${car_width/2 + str_length/2} ${tyre_r}" rpy="0 0 0"/>
-        <axis xyz="0 0 1"/>
-        <limit effort="1000.0" lower="${-str_angle}" upper="${str_angle}" velocity="0.5"/>
-</joint>
-<link name="front_left_steering_link">
-      <parent link="base_link"/>
-        <collision>
-              <xacro:insert_block name="tyre_origin"/>
-                <geometry>
-                 <cylinder length="${str_length}" radius="${str_radius}"/>
-                </geometry>
-        </collision>
-        <visual>
-              <xacro:insert_block name="tyre_origin"/>
-                <geometry>
-                 <cylinder length="${str_length}" radius="${str_radius}"/>
-                </geometry>
-        </visual>
-      <inertial>
-        <origin xyz="0 0 0" rpy="0 0 0"/>
-        <mass value="10.00"/>
-        <inertia
+    </inertial>
+  </link>
+  <!--Left Steering-->
+  <joint name="front_left_steering_joint" type="revolute">
+    <parent link="base_link"/>
+    <child link="front_left_steering_link"/>
+    <origin xyz="${tyre_x} ${car_width/2 + str_length/2} ${tyre_r}" rpy="0 0 0"/>
+    <axis xyz="0 0 1"/>
+    <limit effort="1000.0" lower="${-str_angle}" upper="${str_angle}" velocity="0.5"/>
+  </joint>
+  <link name="front_left_steering_link">
+    <parent link="base_link"/>
+    <collision>
+      <xacro:insert_block name="tyre_origin"/>
+      <geometry>
+        <cylinder length="${str_length}" radius="${str_radius}"/>
+      </geometry>
+    </collision>
+    <visual>
+      <xacro:insert_block name="tyre_origin"/>
+      <geometry>
+        <cylinder length="${str_length}" radius="${str_radius}"/>
+      </geometry>
+    </visual>
+    <inertial>
+      <origin xyz="0 0 0" rpy="0 0 0"/>
+      <mass value="10.00"/>
+      <inertia
           ixx="0.4"  ixy="0.000000"  ixz="0.000000"
           iyy="0.6"  iyz="0.000000"
           izz="0.4"/>
-      </inertial>
-</link>
-<!--Front Right Wheel-->
-<joint name="front_left_wheel_joint" type="continuous">
-      <parent link="front_left_steering_link"/>
-      <child link="front_left_wheel_link"/>
-      <origin xyz="0 ${str_length/2 + tyre_length/2} 0" rpy="0 0 0"/>
-      <axis xyz="0 1 0"/>
-      <dynamics damping="0.1"/>
-      <limit effort="10000" velocity="100" />
-      <joint_properties damping="0.0" friction="0.0" />
-</joint>
-<link name="front_left_wheel_link">
-     <parent link="front_left_wheel_joint"/>
-     <collision>
-	<origin xyz="0 0 0" rpy="${PI/2} 0 0"/>
-        <geometry>
-         <cylinder length="0.229" radius="${tyre_radius}"/>
-        </geometry>
-     </collision>
-     <visual>
+    </inertial>
+  </link>
+  <!--Front Right Wheel-->
+  <joint name="front_left_wheel_joint" type="continuous">
+    <parent link="front_left_steering_link"/>
+    <child link="front_left_wheel_link"/>
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