Commit message: from linux

File: ROS/catkin_ws/src/mercedes/urdf/mercedes.urdf (robot description, URDF)
Before this commit: robot mercedes, 1 links, 0 joints
Links:
- added link fwl, mass 18.5176274523984; collision mesh filename=package://mercedes/meshes/fwl.STL; visual mesh filename=package://mercedes/meshes/fwl.STL
- added link fwr, mass 18.518; collision mesh filename=package://mercedes/meshes/fwr.STL; visual mesh filename=package://mercedes/meshes/fwr.STL
- added link rwl, mass 18.5176264794013; collision mesh filename=package://mercedes/meshes/rwl.STL; visual mesh filename=package://mercedes/meshes/rwl.STL
- added link rwr, mass 18.5176283437402; collision mesh filename=package://mercedes/meshes/rwr.STL; visual mesh filename=package://mercedes/meshes/rwr.STL
- link base_link: mass 0.21541 -> 0.46994
Joints:
- added joint fwl: type continuous, parent base_link, child fwl, origin xyz=0 0 0 rpy=0 0 0, axis 0 -1 0
- added joint fwr: type continuous, parent base_link, child fwr, origin xyz=0 0 0 rpy=0 0 0, axis 0 -1 0
- added joint rwl: type continuous, parent base_link, child rwl, origin xyz=0 0 0 rpy=0 0 0, axis 0 -1 0
- added joint rwr: type continuous, parent base_link, child rwr, origin xyz=0 0 0 rpy=0 0 0, axis 0 -1 0
