Commit message: from linux

File: ROS/catkin_ws/src/dyros_simulator/dyros_simualtor/urdf/HDL-32E.urdf.xacro (robot description, xacro)
@@ -16,5 +16,5 @@
       <visual>
         <geometry>
-          <mesh filename="package://velodyne_description/meshes/HDL32E_base.dae" />
+          <mesh filename="package://dyros_simulator/meshes/HDL32E_base.dae" />
         </geometry>
       </visual>
@@ -40,5 +40,5 @@
         <origin xyz="0 0 -0.09081" rpy="0 0 0" />
         <geometry>
-          <mesh filename="package://velodyne_description/meshes/HDL32E_scan.dae" />
+          <mesh filename="package://dyros_simulator/meshes/HDL32E_scan.dae" />
         </geometry>
       </visual>
@@ -67,5 +67,5 @@
           <range>
             <min>0.1</min>
-            <max>10.0</max>
+            <max>100.0</max>
             <resolution>0.001</resolution>
           </range>

File: ROS/catkin_ws/src/dyros_simulator/dyros_simualtor/urdf/mkz_13_structure.urdf.xacro (robot description, xacro)
@@ -2,5 +2,5 @@
 <!-- created with Phobos 0.7 -->
   <robot name="dbw_mkz" xmlns:xacro="http://www.ros.org/wiki/xacro">
-    <xacro:arg name="dae_file" default="$(find dbw_mkz_description)/meshes/mkz_13/body.dae"/>
+    <xacro:arg name="dae_file" default="$(find dyros_simulator)/meshes/mkz_13/body.dae"/>
     <link name="base_footprint">
     </link>
@@ -21,5 +21,5 @@
         <origin xyz="0.084967 -0.03046 0.350609" rpy="1.570796 0 -3.141593"/>
         <geometry>
-          <mesh filename="package://dbw_mkz_description/meshes/body_collision.stl" scale="0.001 0.001 0.001"/>
+          <mesh filename="package://dyros_simulator/meshes/mkz_13/body.dae" scale="0.001 0.001 0.001"/>
         </geometry>
       </collision>
@@ -68,5 +68,5 @@
         <origin xyz="0 0 -0.043777" rpy="-1.570796 1.570796 0"/>
         <geometry>
-          <mesh filename="package://dbw_mkz_description/meshes/mkz_13/wheel.dae" scale="0.01 0.01 0.01"/>
+          <mesh filename="package://dyros_simulator/meshes/mkz_13/wheel.dae" scale="0.01 0.01 0.01"/>
         </geometry>
         <material name="carpaint_002.001"/>
@@ -88,5 +88,5 @@
         <origin xyz="0 0 0.017382" rpy="-1.570796 -1.570796 0"/>
         <geometry>
-          <mesh filename="package://dbw_mkz_description/meshes/mkz_13/wheel.dae" scale="0.01 0.01 0.01"/>
+          <mesh filename="package://dyros_simulator/meshes/mkz_13/wheel.dae" scale="0.01 0.01 0.01"/>
         </geometry>
         <material name="carpaint_002.003"/>
@@ -108,5 +108,5 @@
         <origin xyz="0 0 -0.019214" rpy="-1.570796 1.570796 0"/>
         <geometry>
-          <mesh filename="package://dbw_mkz_description/meshes/mkz_13/wheel.dae" scale="0.01 0.01 0.01"/>
+          <mesh filename="package://dyros_simulator/meshes/mkz_13/wheel.dae" scale="0.01 0.01 0.01"/>
         </geometry>
         <material name="carpaint_002.002"/>

File: ROS/catkin_ws/src/dyros_simulator/dyros_simualtor/urdf/sick_lms291.urdf.xacro (robot description, xacro)
@@ -4,13 +4,12 @@
   <xacro:property name="sensor_box" value="0.25"/>
   <xacro:macro name="sick_lms291" params="parent name topic *origin">
-    <joint name="sick_lms291_base_mount_joint" type="fixed">
+    <joint name="${name}_base_mount_joint" type="fixed">
       <xacro:insert_block name="origin" />
       <parent link="${parent}"/>
-      <child link="sick_lms291_base_link"/>
+      <child link="${name}_base_link"/>
     </joint>
-    <link name="sick_lms291_base_link">
+    <link name="${name}_base_link">
     </link>
-    <link name="front_laser_link">
-      <parent link="front_laser_joint"/>
+    <link name="${name}">
       <collision>
         <origin xyz="0 0 0" rpy="0 0.0 0"/>
@@ -31,17 +30,17 @@
       </inertial>
     </link>
-    <joint name="front_laser_joint" type="fixed">
+    <joint name="${name}_laser_joint" type="fixed">
       <origin xyz="2.5 0 ${ sensor_box/2}" rpy="0 0 0"/>  <!-- ed: modified-->
       <axis xyz="0 0 1"/>
-      <parent link="sick_lms291_base_link"/>
-      <child link="front_laser_link"/>
+      <parent link="${name}_base_link"/>
+      <child link="${name}"/>
     </joint>
-    <gazebo reference="front_laser_link">
+    <gazebo reference="${name}">
       <mu1>0.6</mu1>
       <mu2>0.5</mu2>
     </gazebo>
     <!-- ed: front laser sensor config code -->
-    <gazebo reference="front_laser_link">
-      <sensor type="ray" name="sick_lms291">
+    <gazebo reference="${name}">
+      <sensor type="ray" name="${name}-sick_lms291">
         <pose>0 0 0 0 0 0</pose>
         <visualize>false</visualize>

File: ROS/catkin_ws/src/dyros_simulator/dyros_simualtor/urdf/vehicle_gazebo.urdf.xacro (robot description, xacro)
@@ -1,5 +1,5 @@
 <?xml version="1.0"?>
 <robot name="mkz_gazebo" xmlns:xacro="http://www.ros.org/wiki/xacro">
-  <xacro:property name="wheel_friction" value="1.2" />
+  <xacro:property name="wheel_friction" value="12" />
   <xacro:arg name="pub_odom" default="false"/>
   <xacro:arg name="pub_tf" default="false"/>

File: ROS/catkin_ws/src/dyros_simulator/dyros_simualtor/urdf/vehicle_sensors.urdf.xacro (robot description, xacro)
@@ -105,11 +105,11 @@
   </xacro:macro>
   <!-- ed: Velodyne sensor added -->
-  <xacro:include filename="$(find velodyne_description)/urdf/HDL-32E.urdf.xacro"/>
-  <HDL-32E parent="base_link" name="/vehicle/velodyne2" topic="/velodyne_points2">
+  <xacro:include filename="$(find dyros_simulator)/urdf/HDL-32E.urdf.xacro"/>
+  <HDL-32E parent="base_link" name="/dyros/velodyne" topic="/velodyne_points">
     <origin xyz="0 0 1.1" rpy="0 0 0" />
   </HDL-32E>
   <!-- ed: sick_laser sensor added -->
-  <xacro:include filename="$(find dbw_mkz_description)/urdf/sick_lms291.urdf.xacro"/>
-  <sick_lms291 parent="base_link" name="/vehicle/front_laser_points" topic="/front_laser_points">
+  <xacro:include filename="$(find dyros_simulator)/urdf/sick_lms291.urdf.xacro"/>
+  <sick_lms291 parent="base_link" name="/dyros/front_laser_points" topic="/front_laser_points">
     <origin xyz="0 0 0" rpy="0 0 0" />
   </sick_lms291>

File: ROS/catkin_ws/src/dyros_simulator/dyros_simualtor/urdf/vehicle_structure.urdf.xacro (robot description, xacro)
@@ -1,4 +1,4 @@
 <?xml version="1.0"?>
 <robot name="dbw_mkz_loader" xmlns:xacro="http://www.ros.org/wiki/xacro">
-  <xacro:include filename="$(find dbw_mkz_description)/urdf/$(arg urdf_model)_structure.urdf.xacro" />
+  <xacro:include filename="$(find dyros_simulator)/urdf/$(arg urdf_model)_structure.urdf.xacro" />
 </robot>
