Commit message: from linux

File: ROS/catkin_ws/src/dyros_simulator/dyros_simualtor/urdf/mkz_13_structure.urdf.xacro (robot description, xacro)
@@ -129,5 +129,6 @@
       <child link="steer_fl"/>
       <axis xyz="0 0 1.0"/>
-      <limit lower="-0.6" upper="0.6" effort="0" velocity="0"/>
+      <!-- ed: 0.6 ==> 0.52 modifed -->
+      <limit lower="-0.52" upper="0.52" effort="0" velocity="0"/>
     </joint>
     <joint name="steer_fr" type="revolute">
@@ -136,5 +137,5 @@
       <child link="steer_fr"/>
       <axis xyz="0 0 1.0"/>
-      <limit lower="-0.6" upper="0.6" effort="0" velocity="0"/>
+      <limit lower="-0.52" upper="0.52" effort="0" velocity="0"/>
     </joint>
     <joint name="wheel_fl" type="continuous">

File: ROS/catkin_ws/src/dyros_simulator/dyros_simualtor/urdf/vehicle_gazebo.urdf.xacro (robot description, xacro)
@@ -1,5 +1,6 @@
 <?xml version="1.0"?>
 <robot name="mkz_gazebo" xmlns:xacro="http://www.ros.org/wiki/xacro">
-  <xacro:property name="wheel_friction" value="12" />
+  <!-- ed: 1.2 is a proper value not to move unnaturally when steering -->
+  <xacro:property name="wheel_friction" value="1.2" />
   <xacro:arg name="pub_odom" default="false"/>
   <xacro:arg name="pub_tf" default="false"/>
