Commit message: from linux

File: ROS/catkin_ws/src/dyros_simulator/dyros_simualtor/urdf/mkz.urdf.xacro (robot description, xacro)
@@ -6,5 +6,5 @@
   <!-- Bolt-on sensors go here -->
   <xacro:include filename="$(find dyros_simulator)/urdf/vehicle_sensors.urdf.xacro" />
-  <xacro:dbw_mkz_camera name="front_camera" parent_link="base_footprint" x="0.6" y="0" z="1.3" roll="0" pitch="0.6" yaw="0" />
+  <!--xacro:dbw_mkz_camera name="front_camera" parent_link="base_footprint" x="0.6" y="0" z="1.3" roll="0" pitch="0.6" yaw="0" /-->
   <xacro:dbw_mkz_gps name="gps" parent_link="base_footprint" x="-0.8" y="0" z="1.45" rate="50.0" ref_lat="45.0" ref_lon="-81.0" />
 </robot>

File: ROS/catkin_ws/src/dyros_simulator/dyros_simualtor/urdf/vehicle_sensors.urdf.xacro (robot description, xacro)
@@ -71,5 +71,5 @@
           <cylinder radius="0.1" length="0.05" />
         </geometry>
-        <material name="white" >
+        <material name="black" >
           <color rgba="1 1 1 1" />
         </material>
@@ -98,6 +98,7 @@
         <ref_lat>${ref_lat}</ref_lat>
         <ref_lon>${ref_lon}</ref_lon>
-        <ant_offset_x>${x}</ant_offset_x>
-        <ant_offset_y>${y}</ant_offset_y>
+        <!-- ed: GPS distance estimation error code -->
+        <ant_offset_x>${x-.5}</ant_offset_x>
+        <ant_offset_y>${y+.5}</ant_offset_y>
         <ant_offset_z>${z}</ant_offset_z>
       </plugin>
